File: hardware/SimpleFlightController.kicad_pcb (KiCad board)
At the start: 2 copper layers, 54.1 x 46.3 mm, 86 parts, among them J1 Screw_Terminal_01x02, J2 Conn_01x03, J3 Conn_01x03, J4 Conn_01x03, J5 Conn_01x03, SW1 TS-1088-AR02016, SW2 TS-1088-AR02016, U1 BQ25883RGER, U2 ICM-45686, U3 STM32F722RETx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

Commit message: SFC v2
Parts:
- added J6: Conn_01x04, Connector_PinHeader_2.54mm:PinHeader_1x04_P2.54mm_Vertical, F.Cu at (139.6, 97.1)
Connections:
- U3 pad 42: unconnected-(U3-PA9-Pad42) -> /CAM_TX
- U3 pad 43: unconnected-(U3-PA10-Pad43) -> /CAM_RX
Routing:
- net /SD_DAT0: track 37.3 -> 37.9 mm
- net /CAM_TX: vias 0 -> 4
- net /CAM_RX: vias 0 -> 4
- net +3.3V: vias 9 -> 11
