File: hardware/SimpleFlightController.kicad_sch (KiCad schematic)
At the start: 86 parts, among them J1 Screw_Terminal_01x02, J2 Conn_01x03, J3 Conn_01x03, J4 Conn_01x03, J5 Conn_01x03, SW1 TS-1088-AR02016, SW2 TS-1088-AR02016, U1 BQ25883RGER, U2 ICM-45686, U3 STM32F722RETx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

Commit message: SFC v2
Parts:
- added J6: Conn_01x04, Connector_PinHeader_2.54mm:PinHeader_1x04_P2.54mm_Vertical, symbol Connector_Generic:Conn_01x04
Connections:
- net +5V: now also J6.1 (Pin_1)
- net GND: now also J6.2 (Pin_2)
- net CAM_TX: now reaches U3.42 (PA9)
- net CAM_TX: now also J6.3 (Pin_3)
- net CAM_RX: now reaches U3.43 (PA10)
- net CAM_RX: now also J6.4 (Pin_4)
- no-connect marks 30 -> 28
